Commit message: Removed schunk_description dependecy, sorted dependencies, added tests for lunch files

File: description/urdf/ftm115.urdf.xacro (robot description, xacro)
@@ -3,19 +3,25 @@
     <xacro:macro name="ati_ftm115" params="parent name *origin">
         <joint name="${name}_base_joint" type="fixed">
-            <insert_block name="origin" />
+            <xacro:insert_block name="origin" />
             <parent link="${parent}"/>
             <child link="${name}_base_link" />
         </joint>
         <link name="${name}_base_link">
-            <xacro:default_inertial/>
+            <inertial>
+                <mass value="0.01" />
+                <origin xyz="0 0 0" />
+                <inertia ixx="0.001" ixy="0.0" ixz="0.0" iyy="0.001" iyz="0.0" izz="0.001" />
+            </inertial>
             <visual>
-                <origin xyz="0 0 0" rpy="0 0 ${-M_PI*3/4}" />
+                <origin xyz="0 0 0" rpy="0 0 ${-pi*3/4}" />
                 <geometry>
                 <mesh filename="package://ati_force_torque/description/meshes/ftm115.stl" scale="0.001 0.001 0.001" />
                 </geometry>
-                <material name="Schunk/DarkGrey" />
+                <material name="DarkGrey">
+                  <color rgba="0.4 0.4 0.4 1.0"/>
+                </material>
             </visual>
             <collision>
-                <origin xyz="0 0 0" rpy="0 0 ${-M_PI*3/4}" />
+                <origin xyz="0 0 0" rpy="0 0 ${-pi*3/4}" />
                 <geometry>
                     <mesh filename="package://ati_force_torque/description/meshes/ftm115.stl" scale="0.001 0.001 0.001" />
@@ -24,19 +30,16 @@
         </link>
         <joint name="${name}_reference_joint" type="fixed">
-            <origin xyz="0 0 ${0.0749-0.01715}" rpy="0 0 ${-M_PI/4}" />
+            <origin xyz="0 0 ${0.0749-0.01715}" rpy="0 0 ${-pi/4}" />
             <parent link="${name}_base_link"/>
             <child link="${name}_reference_link" />
         </joint>
         <link name="${name}_reference_link">
-            <xacro:default_inertial/>
         </link>
         <joint name="${name}_tool_joint" type="fixed">
-            <origin xyz="0 0 0.0749" rpy="0 0 ${-M_PI/12}" />
+            <origin xyz="0 0 0.0749" rpy="0 0 ${-pi/12}" />
             <parent link="${name}_base_link"/>
             <child link="${name}_tool_link" />
         </joint>
-        <link name="${name}_tool_link">
-            <xacro:default_inertial/>
-        </link>
+        <link name="${name}_tool_link"/>
   </xacro:macro>
 </robot>

File: description/urdf/sensor.urdf.xacro (robot description, xacro)
@@ -2,7 +2,4 @@
 <robot xmlns:xacro="http://www.ros.org/wiki/xacro"
        name="ati_ftm115" >
-  <!-- common stuff -->
-  <xacro:include filename="$(find schunk_description)/urdf/common.xacro" />
-  <xacro:include filename="$(find schunk_description)/urdf/materials.urdf.xacro" />
   <!-- ati ftm115 -->
   <xacro:include filename="$(find ati_force_torque)/description/urdf/ftm115.urdf.xacro" />

Commit message: changes for simulation.need to be cleaned

File: description/urdf/ftm115.urdf.xacro (robot description, xacro)
@@ -1,7 +1,10 @@
 <?xml version="1.0"?>
 <robot xmlns:xacro="http://www.ros.org/wiki/xacro">
+    <xacro:include filename="$(find ati_force_torque)/description/urdf/ftm115.transmission.xacro" />
+    <xacro:include filename="$(find ati_force_torque)/description/urdf/ftm115.gazebo.xacro" />
     <xacro:macro name="ati_ftm115" params="parent name *origin">
-        <joint name="${name}_base_joint" type="fixed">
+        <joint name="${name}_base_joint" type="continuous">
             <xacro:insert_block name="origin" />
+            <origin xyz="-0.348 0 0.96" rpy="0 0 0" />
             <parent link="${parent}"/>
             <child link="${name}_base_link" />
@@ -10,5 +13,5 @@
             <xacro:default_inertial/>
             <visual>
-                <origin xyz="0 0 0" rpy="0 0 ${-M_PI*3/4}" />
+                <origin xyz="0 0 -0.4" rpy="0 0 0" />
                 <geometry>
                 <mesh filename="package://ati_force_torque/description/meshes/ftm115.stl" scale="0.001 0.001 0.001" />
@@ -23,6 +26,6 @@
             </collision>
         </link>
-        <joint name="${name}_reference_joint" type="fixed">
-            <origin xyz="0 0 ${0.0749-0.01715}" rpy="0 0 ${-M_PI/4}" />
+        <joint name="${name}_reference_joint" type="continuous">
+            <origin xyz="0 0 0" rpy="2.991 -0.918 -3.067" />
             <parent link="${name}_base_link"/>
             <child link="${name}_reference_link" />
@@ -31,5 +34,5 @@
             <xacro:default_inertial/>
         </link>
-        <joint name="${name}_tool_joint" type="fixed">
+        <!--<joint name="${name}_tool_joint" type="fixed">
             <origin xyz="0 0 0.0749" rpy="0 0 ${-M_PI/12}" />
             <parent link="${name}_base_link"/>
@@ -38,5 +41,8 @@
         <link name="${name}_tool_link">
             <xacro:default_inertial/>
-        </link>
+        </link>-->
+        <xacro:fts_gazebo_ref_link parent="${name}"  />
+        <xacro:fts_gazebo_base_link parent="${name}"  />
+        <xacro:fts_transmission parent="${name}"  />
   </xacro:macro>
 </robot>

Commit message: merged master branch with raw_with_fts

File: description/urdf/ftm115.urdf.xacro (robot description, xacro)
@@ -11,20 +11,15 @@
         </joint>
         <link name="${name}_base_link">
-            <inertial>
-                <mass value="0.01" />
-                <origin xyz="0 0 0" />
-                <inertia ixx="0.001" ixy="0.0" ixz="0.0" iyy="0.001" iyz="0.0" izz="0.001" />
-            </inertial>
+            <xacro:default_inertial/>
             <visual>
 <!--<<<<<<< HEAD
-                <origin xyz="0 0 0" rpy="0 0 ${-pi*3/4}" />
-                =======-->
+      <origin xyz="0 0 0" rpy="0 0 ${-pi*3/4}" />
+=======
+-->
                 <origin xyz="0 0 -0.4" rpy="0 0 0" />
                 <geometry>
                 <mesh filename="package://ati_force_torque/description/meshes/ftm115.stl" scale="0.001 0.001 0.001" />
                 </geometry>
-                <material name="DarkGrey">
-                  <color rgba="0.4 0.4 0.4 1.0"/>
-                </material>
+                <material name="Schunk/DarkGrey" />
             </visual>
             <collision>
@@ -38,5 +33,6 @@
         <joint name="${name}_reference_joint" type="fixed">
             <origin xyz="0 0 ${0.0749-0.01715}" rpy="0 0 ${-pi/4}" />
-        =======-->
+=======
+-->
         <joint name="${name}_reference_joint" type="continuous">
             <origin xyz="0 0 0" rpy="2.991 -0.918 -3.067" />
@@ -45,22 +41,17 @@
         </joint>
         <link name="${name}_reference_link">
+            <xacro:default_inertial/>
         </link>
 <!--
-<<<<<<< HEAD
+HEAD
         <joint name="${name}_tool_joint" type="fixed">
             <origin xyz="0 0 0.0749" rpy="0 0 ${-pi/12}" />
-=======
-        <joint name="${name}_tool_joint" type="fixed">
-            <origin xyz="0 0 0.0749" rpy="0 0 ${-pi/12}" />
->>>>>>> raw_with_fts
             <parent link="${name}_base_link"/>
             <child link="${name}_tool_link" />
         </joint>
-<<<<<<< HEAD
-        <link name="${name}_tool_link"/>
-=======
         <link name="${name}_tool_link">
             <xacro:default_inertial/>
-        </link>-->
+        </link>
+-->
         <xacro:fts_gazebo_ref_link parent="${name}"  />
         <xacro:fts_gazebo_base_link parent="${name}"  />

Commit message: small changes in urdf

File: description/urdf/ftm115.urdf.xacro (robot description, xacro)
@@ -4,7 +4,6 @@
     <xacro:include filename="$(find ati_force_torque)/description/urdf/ftm115.gazebo.xacro" />
     <xacro:macro name="ati_ftm115" params="parent name *origin">
-        <joint name="${name}_base_joint" type="continuous">
+        <joint name="${name}_base_joint" type="fixed">
             <xacro:insert_block name="origin" />
-            <origin xyz="-0.348 0 0.96" rpy="0 0 0" />
             <parent link="${parent}"/>
             <child link="${name}_base_link" />
@@ -13,5 +12,5 @@
             <xacro:default_inertial/>
             <visual>
-                <origin xyz="0 0 -0.4" rpy="0 0 0" />
+                <origin xyz="0 0 0" rpy="0 0 0" />
                 <geometry>
                 <mesh filename="package://ati_force_torque/description/meshes/ftm115.stl" scale="0.001 0.001 0.001" />
@@ -27,5 +26,5 @@
         </link>
         <joint name="${name}_reference_joint" type="continuous">
-            <origin xyz="0 0 0" rpy="2.991 -0.918 -3.067" />
+            <origin xyz="0 0 0" rpy="0.0 0.0 -2.216 " />
             <parent link="${name}_base_link"/>
             <child link="${name}_reference_link" />
@@ -34,12 +33,4 @@
             <xacro:default_inertial/>
         </link>
-        <!--<joint name="${name}_tool_joint" type="fixed">
-            <origin xyz="0 0 0.0749" rpy="0 0 ${-M_PI/12}" />
-            <parent link="${name}_base_link"/>
-            <child link="${name}_tool_link" />
-        </joint>
-        <link name="${name}_tool_link">
-            <xacro:default_inertial/>
-        </link>-->
         <xacro:fts_gazebo_ref_link parent="${name}"  />
         <xacro:fts_gazebo_base_link parent="${name}"  />

Commit message: some more changes for PR

File: description/urdf/ftm115.urdf.xacro (robot description, xacro)
@@ -16,5 +16,7 @@
                 <mesh filename="package://ati_force_torque/description/meshes/ftm115.stl" scale="0.001 0.001 0.001" />
                 </geometry>
-                <material name="Schunk/DarkGrey" />
+                <material name="DarkGrey">
+                    <color rgba="0.4 0.4 0.4 1.0"/>
+                </material>
             </visual>
             <collision>

Commit message: changes for PR

File: description/urdf/ftm115.urdf.xacro (robot description, xacro)
@@ -1,6 +1,4 @@
 <?xml version="1.0"?>
 <robot xmlns:xacro="http://www.ros.org/wiki/xacro">
-    <xacro:include filename="$(find ati_force_torque)/description/urdf/ftm115.transmission.xacro" />
-    <xacro:include filename="$(find ati_force_torque)/description/urdf/ftm115.gazebo.xacro" />
     <xacro:macro name="ati_ftm115" params="parent name *origin">
         <joint name="${name}_base_joint" type="fixed">
@@ -10,12 +8,16 @@
         </joint>
         <link name="${name}_base_link">
-            <xacro:default_inertial/>
+            <inertial>
+                <mass value="0.01" />
+                <origin xyz="0 0 0" />
+                <inertia ixx="0.001" ixy="0.0" ixz="0.0" iyy="0.001" iyz="0.0" izz="0.001" />
+            </inertial>
             <visual>
-                <origin xyz="0 0 0" rpy="0 0 0" />
+                <origin xyz="0 0 0" rpy="0 0 ${-pi*3/4}" />
                 <geometry>
                 <mesh filename="package://ati_force_torque/description/meshes/ftm115.stl" scale="0.001 0.001 0.001" />
                 </geometry>
                 <material name="DarkGrey">
-                    <color rgba="0.4 0.4 0.4 1.0"/>
+                  <color rgba="0.4 0.4 0.4 1.0"/>
                 </material>
             </visual>
@@ -27,15 +29,17 @@
             </collision>
         </link>
-        <joint name="${name}_reference_joint" type="continuous">
-            <origin xyz="0 0 0" rpy="0.0 0.0 -2.216 " />
+        <joint name="${name}_reference_joint" type="fixed">
+            <origin xyz="0 0 ${0.0749-0.01715}" rpy="0 0 ${-pi/4}" />
             <parent link="${name}_base_link"/>
             <child link="${name}_reference_link" />
         </joint>
         <link name="${name}_reference_link">
-            <xacro:default_inertial/>
         </link>
-        <xacro:fts_gazebo_ref_link parent="${name}"  />
-        <xacro:fts_gazebo_base_link parent="${name}"  />
-        <xacro:fts_transmission parent="${name}"  />
+        <joint name="${name}_tool_joint" type="fixed">
+            <origin xyz="0 0 0.0749" rpy="0 0 ${-pi/12}" />
+            <parent link="${name}_base_link"/>
+            <child link="${name}_tool_link" />
+        </joint>
+        <link name="${name}_tool_link"/>
   </xacro:macro>
 </robot>

File: description/urdf/fts.gazebo.xacro (robot description, xacro)
@@ -13,3 +13,9 @@
     </gazebo>
   </xacro:macro>
+   <xacro:macro name="fts_gazebo_ref_joint" params="parent ">
+    <gazebo reference="${parent}_reference_joint">
+      <gravity>true</gravity>
+      <self_collide>false</self_collide>
+    </gazebo>
+  </xacro:macro>
 </robot>
