Commit message: small change for sensor simulation

File: description/urdf/sensor_mini58.urdf.xacro (robot description, xacro)
@@ -4,4 +4,12 @@
   <xacro:if value="$(arg sim)">
 	  <xacro:include filename="$(find ati_force_torque)/description/urdf/macros/mini58_sim.urdf.xacro" />
+      <!-- Used for sensor simulation -->
+    <xacro:macro name="default_inertial">
+        <inertial>
+            <mass value="0.01"/>
+            <origin xyz="0 0 0"/>
+            <inertia ixx="0.001" ixy="0.0" ixz="0.0" iyy="0.001" iyz="0.0" izz="0.001" />
+        </inertial>
+    </xacro:macro>
   </xacro:if>
   <xacro:unless value="$(arg sim)">
@@ -10,5 +18,5 @@
   <!-- Used for fixing sensor to Gazebo -->
   <link name="base_link"/>
-  <!-- sensor -->
+<!-- sensor -->
   <xacro:ati_mini58 name="fts" parent="base_link">
       <origin xyz="0 0 0" rpy="0 0 0" />
