Commit message: changes in urdf file for correct description when using sensor with sr2

File: description/urdf/macros/mini58.urdf.xacro (robot description, xacro)
@@ -27,5 +27,5 @@
             </collision>
         </link>
-        <joint name="${name}_tool_joint" type="fixed">
+<!--        <joint name="${name}_tool_joint" type="fixed">
             <origin xyz="0 0 0.03" rpy="0 0 0" />
             <parent link="${name}_base_link"/>
@@ -33,7 +33,8 @@
         </joint>
         <link name="${name}_tool_link"/>
+-->
         <joint name="${name}_reference_joint" type="fixed">
-            <origin xyz="0 0 0" rpy="0 0 0" />
-            <parent link="${name}_tool_link"/>
+            <origin xyz="0 0 0" rpy="0 0 -2.22068070" />
+            <parent link="${name}_base_link"/>
             <child link="${name}_reference_link" />
         </joint>

File: description/urdf/macros/mini58_sim.urdf.xacro (robot description, xacro)
@@ -1,4 +1,5 @@
 <?xml version="1.0"?>
 <robot xmlns:xacro="http://www.ros.org/wiki/xacro">
+    <xacro:include filename="$(find ati_force_torque)/description/urdf/fts.transmission.xacro" />
     <xacro:macro name="ati_mini58" params="parent name *origin">
 <!--         Shift for -30 -90 -->
@@ -41,9 +42,8 @@
             <child link="${name}_tool_link" />
         </joint>
-       <joint name="${name}_reference_joint" type="revolute">
+       <joint name="${name}_reference_joint" type="fixed">
             <origin xyz="0 0 0" rpy="0 0 0" />
             <parent link="${name}_tool_link"/>
             <child link="${name}_reference_link" />
-            <limit effort="0.0" lower="0.0" upper="0.0" velocity="0.0"/>
         </joint>
         <xacro:fts_transmission parent="${name}"  />

Commit message: moved ati ft for sr2 to sr2_bringup

File: description/urdf/macros/mini58.urdf.xacro (robot description, xacro)
@@ -27,5 +27,5 @@
             </collision>
         </link>
-<!--        <joint name="${name}_tool_joint" type="fixed">
+        <joint name="${name}_tool_joint" type="fixed">
             <origin xyz="0 0 0.03" rpy="0 0 0" />
             <parent link="${name}_base_link"/>
@@ -33,9 +33,8 @@
         </joint>
         <link name="${name}_tool_link"/>
--->
         <joint name="${name}_reference_joint" type="fixed">
-            <origin xyz="0 0 0" rpy="0 0 -2.22068070" />
+            <origin xyz="0 0 0" rpy="0 0 0" />
             <parent link="${name}_base_link"/>
-            <child link="${name}_reference_link" />
+            <child link="${name}_tool_link" />
         </joint>
         <link name="${name}_reference_link">

File: description/urdf/macros/mini58_sim.urdf.xacro (robot description, xacro)
@@ -42,8 +42,9 @@
             <child link="${name}_tool_link" />
         </joint>
-       <joint name="${name}_reference_joint" type="fixed">
+       <joint name="${name}_reference_joint" type="revolute">
             <origin xyz="0 0 0" rpy="0 0 0" />
             <parent link="${name}_tool_link"/>
             <child link="${name}_reference_link" />
+	    <limit effort="0.0" lower="0.0" upper="0.0" velocity="0.0"/>
         </joint>
         <xacro:fts_transmission parent="${name}"  />

File: description/urdf/sensor_mini58.urdf.xacro (robot description, xacro)
@@ -1,7 +1,11 @@
 <?xml version="1.0"?>
-<robot xmlns:xacro="http://www.ros.org/wiki/xacro"
-       name="ati_mini58" >
+<robot xmlns:xacro="http://www.ros.org/wiki/xacro" name="ati_mini58" >
   <!-- ati_mini58 -->
-  <xacro:include filename="$(find ati_force_torque)/description/urdf/macros/mini58.urdf.xacro" />
+  <xacro:if value="$(arg sim)">
+	  <xacro:include filename="$(find ati_force_torque)/description/urdf/macros/mini58_sim.urdf.xacro" />
+  </xacro:if>
+  <xacro:unless value="$(arg sim)">
+	  <xacro:include filename="$(find ati_force_torque)/description/urdf/macros/mini58.urdf.xacro" />
+  </xacro:unless>
   <!-- Used for fixing sensor to Gazebo -->
   <link name="base_link"/>

Commit message: undone small change in urdf

File: description/urdf/macros/mini58.urdf.xacro (robot description, xacro)
@@ -35,6 +35,6 @@
         <joint name="${name}_reference_joint" type="fixed">
             <origin xyz="0 0 0" rpy="0 0 0" />
-            <parent link="${name}_base_link"/>
-            <child link="${name}_tool_link" />
+            <parent link="${name}_tool_link"/>
+            <child link="${name}_reference_link" />
         </joint>
         <link name="${name}_reference_link">
