Commit message: Raw with fts (#18)
* Removed dependecy on schunk_description (#6)

* Removed dependecy on schunk_description

* Added xacro dependency

* changes for working raw with fts

* some changes for namespace read

* rosparam working

* added cs calibration params

* added necessary code for simulation

* changes for simulation.need to be cleaned

* changes in fthandle_sim

* deleted prints

* merged master branch with raw_with_fts

* small changes in urdf

* compatibility changes for iirob_fitlers

* Use c++11 and update .travis

* Update .travis.rosinstall

* Updated compile files and some Sim files headers

* made some changes

* some more changes for PR

* changes for PR

* changed in fts.gazebo

* changes for PR

* changes for PR and added sim parameter

* changes for working correctly with rosparam_handler

* changes to work correctly with rosparam and real raw with fts

* changes for working with real sensor and simulation

* not depending on own rosparam_handler anymore

* chages for simulation of sensor

* using teleop not cob_teleop anymore

* remapped to cmd_force

* changed default values for easier debugging

* small changes

* changes to use unchanged sensor_offsets

* added realtime publisher and working with iirob_led

* changes to work with iirob led

* some changes to work with rt publisher and iirob_led after test

* changes for working with iirob filters after changing to plugin

* changes in urdf file for correct description when using sensor with sr2

* changes to work with filters pluginlib

* moved ati ft for sr2 to sr2_bringup

* undone small change in urdf

* small change for sensor simulation

* Update package.xml

* Update package.xml

* Removed iirob_led dependency.

* working branch with iirob_filters

* changes to work with wrench stamped as template

* changes to work with iirob_filters moving mean filter

* use rosparam handler for gravity compensator

* changes to work with filters

* Update sensor_mini58.urdf.xacro

* Update driver_sim.launch

File: description/urdf/macros/mini58_sim.urdf.xacro (robot description, xacro)
@@ -1,4 +1,5 @@
 <?xml version="1.0"?>
 <robot xmlns:xacro="http://www.ros.org/wiki/xacro">
+    <xacro:include filename="$(find ati_force_torque)/description/urdf/fts.transmission.xacro" />
     <xacro:macro name="ati_mini58" params="parent name *origin">
 <!--         Shift for -30 -90 -->

File: description/urdf/sensor_mini58.urdf.xacro (robot description, xacro)
@@ -1,10 +1,23 @@
 <?xml version="1.0"?>
-<robot xmlns:xacro="http://www.ros.org/wiki/xacro"
-       name="ati_mini58" >
+<robot xmlns:xacro="http://www.ros.org/wiki/xacro" name="ati_mini58" >
+  <xacro:arg name="sim" default="false"/>
   <!-- ati_mini58 -->
-  <xacro:include filename="$(find ati_force_torque)/description/urdf/macros/mini58.urdf.xacro" />
+  <xacro:if value="$(arg sim)">
+	  <xacro:include filename="$(find ati_force_torque)/description/urdf/macros/mini58_sim.urdf.xacro" />
+      <!-- Used for sensor simulation -->
+    <xacro:macro name="default_inertial">
+        <inertial>
+            <mass value="0.01"/>
+            <origin xyz="0 0 0"/>
+            <inertia ixx="0.001" ixy="0.0" ixz="0.0" iyy="0.001" iyz="0.0" izz="0.001" />
+        </inertial>
+    </xacro:macro>
+  </xacro:if>
+  <xacro:unless value="$(arg sim)">
+	  <xacro:include filename="$(find ati_force_torque)/description/urdf/macros/mini58.urdf.xacro" />
+  </xacro:unless>
   <!-- Used for fixing sensor to Gazebo -->
   <link name="base_link"/>
-  <!-- sensor -->
+<!-- sensor -->
   <xacro:ati_mini58 name="fts" parent="base_link">
       <origin xyz="0 0 0" rpy="0 0 0" />
